Commit message: Use fixed-standing planar pose control for Go2 application simulation

File: gazebo/robots/go2/go2_tinynav.xacro (robot description, xacro)
@@ -9,4 +9,7 @@
      -topic path drops every sensor pose). -->
 <robot name="go2_tinynav" xmlns:xacro="http://ros.org/wiki/xacro">
+  <xacro:arg name="kinematic" default="false"/>
+  <xacro:property name="kinematic" value="$(arg kinematic)"/>
+  <xacro:property name="stand_angle" value="${acos(0.25 / 0.426)}"/>
   <xacro:arg name="robot_name" default="robot1"/>
   <!-- absolute path of ros_control.yaml, passed by spawn.sh:
@@ -95,5 +98,5 @@
        hip-axis limit signs and the inertial off-diagonal signs. -->
   <xacro:macro name="leg" params="name mirror front_hind">
-    <joint name="${name}_hip_joint" type="revolute">
+    <joint name="${name}_hip_joint" type="${'fixed' if kinematic else 'revolute'}">
       <origin rpy="0 0 0" xyz="${front_hind*leg_offset_x} ${mirror*leg_offset_y} 0"/>
       <parent link="trunk"/>
@@ -131,6 +134,6 @@
       </inertial>
     </link>
-    <joint name="${name}_upper_leg_joint" type="revolute">
-      <origin rpy="0 0 0" xyz="0 ${thigh_offset*mirror} 0"/>
+    <joint name="${name}_upper_leg_joint" type="${'fixed' if kinematic else 'revolute'}">
+      <origin rpy="0 ${stand_angle if kinematic else 0} 0" xyz="0 ${thigh_offset*mirror} 0"/>
       <parent link="${name}_hip_link"/>
       <child link="${name}_upper_leg_link"/>
@@ -162,6 +165,6 @@
       </inertial>
     </link>
-    <joint name="${name}_lower_leg_joint" type="revolute">
-      <origin rpy="0 0 0" xyz="0 0 ${-thigh_length}"/>
+    <joint name="${name}_lower_leg_joint" type="${'fixed' if kinematic else 'revolute'}">
+      <origin rpy="0 ${-2*stand_angle if kinematic else 0} 0" xyz="0 0 ${-thigh_length}"/>
       <parent link="${name}_upper_leg_link"/>
       <child link="${name}_lower_leg_link"/>
@@ -369,4 +372,5 @@
     </sensor>
   </gazebo>
+  <xacro:unless value="${kinematic}">
   <gazebo>
     <plugin name="gz_ros2_control::GazeboSimROS2ControlPlugin" filename="libign_ros2_control-system.so">
@@ -394,4 +398,8 @@
     <xacro:rc_joint name="rh_lower_leg_joint" init="-1.887"/>
   </ros2_control>
+  </xacro:unless>
+  <xacro:if value="${kinematic}">
+    <gazebo><static>true</static></gazebo>
+  </xacro:if>
   <!-- contact surfaces -->
   <gazebo reference="trunk">

Commit message: Add rear Go2 sensor rig and synchronized Looper output

File: gazebo/robots/go2/go2_tinynav.xacro (robot description, xacro)
@@ -277,5 +277,5 @@
   <xacro:property name="head_z" value="0.09"/>
   <xacro:property name="cam_y" value="0.0255"/>
-  <xacro:macro name="sensor_link" params="name x y z">
+  <xacro:macro name="sensor_link" params="name x y z yaw:=0">
     <!-- NO visual: a visual near the camera origin would be rendered by the
          camera itself (inside its own bounding mesh) -->
@@ -287,5 +287,5 @@
     </link>
     <joint name="${name}_joint" type="fixed">
-      <origin xyz="${x} ${y} ${z}" rpy="0 0 0"/>
+      <origin xyz="${x} ${y} ${z}" rpy="0 0 ${yaw}"/>
       <!-- the head rides the trunk: base_link is the ground-level model
            origin and would put the sensors underground -->
@@ -337,4 +337,23 @@
     </gazebo>
   </xacro:macro>
+  <gazebo reference="rear_infra1_link">
+    <sensor name="rear_depth" type="depth_camera">
+      <pose>0 0 0 0 0 0</pose>
+      <camera>
+        <horizontal_fov>1.5708</horizontal_fov>
+        <image><width>544</width><height>480</height><format>R_FLOAT32</format></image>
+        <clip><near>0.1</near><far>15</far></clip>
+      </camera>
+      <always_on>1</always_on>
+      <update_rate>15</update_rate>
+      <topic>/sim/rear/depth</topic>
+    </sensor>
+  </gazebo>
+  <xacro:sensor_link name="rear_infra1" x="-${head_x}" y="-${cam_y}" z="${head_z}" yaw="${PI}"/>
+  <xacro:gz_camera name="rear_infra1" topic="/camera/rear/infra1/image_rect_raw" format="L8"/>
+  <xacro:sensor_link name="rear_infra2" x="-${head_x}" y="${cam_y}" z="${head_z}" yaw="${PI}"/>
+  <xacro:gz_camera name="rear_infra2" topic="/camera/rear/infra2/image_rect_raw" format="L8"/>
+  <xacro:sensor_link name="rear_color" x="-${head_x}" y="0" z="${head_z}" yaw="${PI}"/>
+  <xacro:gz_camera name="rear_color" topic="/camera/rear/color/image_raw" format="RGB_INT8"/>
   <gazebo reference="camera_infra1_link">
     <sensor name="camera_depth" type="depth_camera">
@@ -367,4 +386,16 @@
       <visualize>true</visualize>
       <topic>/camera/camera/imu</topic>
+      <!-- identity translation, same lumping reason as the cameras; the RPY
+           stays: it is the camera-convention rotation (body Z = forward) -->
+      <pose>0 0 0 1.5708 3.14159 1.5708</pose>
+    </sensor>
+  </gazebo>
+  <xacro:sensor_link name="rear_imu" x="-0.15" y="0" z="${head_z}" yaw="${PI}"/>
+  <gazebo reference="rear_imu_link">
+    <sensor name="rear_imu" type="imu">
+      <always_on>1</always_on>
+      <update_rate>200</update_rate>
+      <visualize>true</visualize>
+      <topic>/camera/rear/imu</topic>
       <!-- identity translation, same lumping reason as the cameras; the RPY
            stays: it is the camera-convention rotation (body Z = forward) -->
